File: supervision/supervision.sch (KiCad schematic (older format))
At the start: 8 parts, among them J1 Conn_01x01, J2 Conn_01x01, SW1 SW_DIP_x05, U1 SST39SF040, U2 SV_CART

Commit message: Added megadrive and .kicad_mod files, cleaned up supervision files
Parts:
- U2: symbol SV_CART-RESCUE-supervision -> SV_CART
Changed lines of the file:
@@
 EESchema Schematic File Version 2
-LIBS:supervision-rescue
 LIBS:power
 LIBS:device
@@
 $EndComp
 $Comp
-L SV_CART-RESCUE-supervision U2
+L SV_CART U2
 U 1 1 5A2D579C
 P 6650 1950
