File: eeprom_writer/eeprom_writer.kicad_pcb (KiCad board)
At the start: 2 copper layers, 40 x 40 mm, 16 parts, among them J1 USB_OTG, U1 SST39SF040, U2 74HC595, U3 74HC595, U4 ATMEGA8U2-AU, Y1 12MHz

Commit message: Updated MD, SV, Writer; added GB
Parts:
- added REF**: Socket_Strip_Straight_1x04_Pitch2.54mm, Socket_Strips:Socket_Strip_Straight_1x04_Pitch2.54mm, F.Cu at (107.3, 76.7)
- moved C6 5.47 mm to (112.2, 84.2)
- moved U3 4.91 mm to (116.4, 80.3)
Routing:
- net Net-(U2-Pad11): track 35.0 -> 39.1 mm
- net Net-(U2-Pad12): track 36.3 -> 40.3 mm
- net /A0_: track 25.5 -> 21.8 mm
- net /A1_: track 17.1 -> 13.8 mm
- net /A2_: track 15.5 -> 12.5 mm
- net /A3_: track 13.9 -> 11.7 mm
- net /A4_: track 12.4 -> 11.1 mm
- net /A7_: track 8.17 -> 9.09 mm
- net +5V: track 80.7 -> 81.4 mm, vias 6 -> 7
- net /A5_: track 10.9 -> 10.4 mm
- net Net-(U3-Pad14): track 25.7 -> 26.0 mm, vias 6 -> 4
