File: megadrive/megadrive.kicad_pcb (KiCad board)
At the start: 2 copper layers, 82.3 x 55.4 mm, 7 parts, among them SW1 SW_DIP_x02, U1 MD_CART, U2 SST39SF040, U3 SST39SF040, U4 FM1808B-SG

Commit message: Updated MD, SV, Writer; added GB
Routing:
- net /A10: track 105.0 -> 140.6 mm
- net /A4: track 113.5 -> 115.5 mm
- net /A6: track 79.1 -> 80.7 mm
- net /A18: track 88.8 -> 90.4 mm
- net //OE: track 90.7 -> 92.2 mm
- net /A3: track 80.8 -> 82.3 mm
- net Net-(SW1-Pad1): track 29.9 -> 31.0 mm
- net /A11: track 94.9 -> 96.0 mm
- net /A12: track 91.2 -> 92.1 mm
- net /A19: track 91.9 -> 92.6 mm
- net /A9: track 115.6 -> 114.8 mm
- net /D9: track 63.8 -> 64.3 mm
